Commit message: Worked on integrating SNS.  It works, but need to fine tune the dropping of the object, as well as remove the repressurization of the grasper at the end.  Need to set target and goal position to be dynamic based on user input.

File: Testing/combined.urdf (robot description, URDF)
Before this commit: robot GantryAssembly_NoGrasper, 15 links, 14 joints
Links:
- link BasePlate: geometry collision mesh filename=C:\Users\SmorgasBORG\Documents\GitHub\FRR-Software-Interfac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 scale=1.00000 1.00000 1.00000; visual mesh filename=C:\Users\SmorgasBORG\Documents\GitHub\FRR-Software-Interfac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 scale=1.00000 1.00000 1.00000
- link CylinderCons: geometry collision mesh filename=C:\Users\SmorgasBORG\Documents\GitHub\FRR-Software-Interfac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 scale=1.00000 1.00000 1.00000; visual mesh filename=C:\Users\SmorgasBORG\Documents\GitHub\FRR-Software-Interfac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 scale=1.00000 1.00000 1.00000
- link GrasperBase: geometry collision mesh filename=C:\Users\SmorgasBORG\Documents\GitHub\FRR-Software-Interfac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 scale=1.00000 1.00000 1.00000; visual mesh filename=C:\Users\SmorgasBORG\Documents\GitHub\FRR-Software-Interfac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 scale=1.00000 1.00000 1.00000
- link LeftUpright: geometry collision mesh filename=C:\Users\SmorgasBORG\Documents\GitHub\FRR-Software-Interfac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 scale=1.00000 1.00000 1.00000; visual mesh filename=C:\Users\SmorgasBORG\Documents\GitHub\FRR-Software-Interfac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 scale=1.00000 1.00000 1.00000
- link ObjectBase: geometry collision mesh filename=C:\Users\SmorgasBORG\Documents\GitHub\FRR-Software-Interfac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 scale=1.00000 1.00000 1.00000; visual mesh filename=C:\Users\SmorgasBORG\Documents\GitHub\FRR-Software-Interfac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 scale=1.00000 1.00000 1.00000
- link RightUpright: geometry collision mesh filename=C:\Users\SmorgasBORG\Documents\GitHub\FRR-Software-Interfac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 scale=1.00000 1.00000 1.00000; visual mesh filename=C:\Users\SmorgasBORG\Documents\GitHub\FRR-Software-Interfac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 scale=1.00000 1.00000 1.00000
- link SoftJaw1: geometry collision mesh filename=C:\Users\SmorgasBORG\Documents\GitHub\FRR-Software-Interfac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 scale=1.00000 1.00000 1.00000; visual mesh filename=C:\Users\SmorgasBORG\Documents\GitHub\FRR-Software-Interfac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 scale=1.00000 1.00000 1.00000
- link SoftJaw2: geometry collision mesh filename=C:\Users\SmorgasBORG\Documents\GitHub\FRR-Software-Interfac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 scale=1.00000 1.00000 1.00000; visual mesh filename=C:\Users\SmorgasBORG\Documents\GitHub\FRR-Software-Interfac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 scale=1.00000 1.00000 1.00000
- link SoftJaw3: geometry collision mesh filename=C:\Users\SmorgasBORG\Documents\GitHub\FRR-Software-Interfac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 scale=1.00000 1.00000 1.00000; visual mesh filename=C:\Users\SmorgasBORG\Documents\GitHub\FRR-Software-Interfac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 scale=1.00000 1.00000 1.00000
- link SoftSupport1: geometry collision mesh filename=C:\Users\SmorgasBORG\Documents\GitHub\FRR-Software-Interfac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 scale=1.00000 1.00000 1.00000; visual mesh filename=C:\Users\SmorgasBORG\Documents\GitHub\FRR-Software-Interfac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 scale=1.00000 1.00000 1.00000
- link SoftSupport2: geometry collision mesh filename=C:\Users\SmorgasBORG\Documents\GitHub\FRR-Software-Interfac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 scale=1.00000 1.00000 1.00000; visual mesh filename=C:\Users\SmorgasBORG\Documents\GitHub\FRR-Software-Interfac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 scale=1.00000 1.00000 1.00000
- link SoftSupport3: geometry collision mesh filename=C:\Users\SmorgasBORG\Documents\GitHub\FRR-Software-Interfac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 scale=1.00000 1.00000 1.00000; visual mesh filename=C:\Users\SmorgasBORG\Documents\GitHub\FRR-Software-Interfac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 scale=1.00000 1.00000 1.00000
- link ZBar: geometry collision mesh filename=C:\Users\SmorgasBORG\Documents\GitHub\FRR-Software-Interfac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 scale=1.00000 1.00000 1.00000; visual mesh filename=C:\Users\SmorgasBORG\Documents\GitHub\FRR-Software-Interfac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 scale=1.00000 1.00000 1.00000
- link base_link: geometry collision mesh filename=C:\Users\SmorgasBORG\Documents\GitHub\FRR-Software-Interfac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 scale=1.00000 1.00000 1.00000; visual mesh filename=C:\Users\SmorgasBORG\Documents\GitHub\FRR-Software-Interfac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 scale=1.00000 1.00000 1.00000
- link base_link_gantry: geometry collision mesh filename=C:\Users\SmorgasBORG\Documents\GitHub\FRR-Software-Interfac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 scale=1.00000 1.00000 1.00000; visual mesh filename=C:\Users\SmorgasBORG\Documents\GitHub\FRR-Software-Interfac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 scale=1.00000 1.00000 1.00000
Joints:
- joint BCC: limit lower=-0.50000 upper=0.50000 effort=1000.0 velocity=0.5 -> lower=-2.50000 upper=2.50000 effort=0.00000 velocity=0.00000
- joint BasePlateJoint: limit lower=-0.50000 upper=0.50000 effort=1000.0 velocity=0.5 -> lower=-0.30000 upper=0.30000 effort=0.00000 velocity=0.00000
- joint GrasperBase: limit lower=-0.50000 upper=0.50000 effort=1000.0 velocity=0.5 -> lower=-0.20000 upper=0.20000 effort=0.00000 velocity=0.00000
- joint LinearJaw1: limit lower=-0.50000 upper=0.50000 effort=1000.0 velocity=0.5 -> lower=0.00000 upper=0.02800 effort=0.00000 velocity=0.00000
- joint LinearJaw2: limit lower=-0.50000 upper=0.50000 effort=1000.0 velocity=0.5 -> lower=0.00000 upper=0.02800 effort=0.00000 velocity=0.00000
- joint LinearJaw3: limit lower=-0.50000 upper=0.50000 effort=1000.0 velocity=0.5 -> lower=0.00000 upper=0.02800 effort=0.00000 velocity=0.00000
- joint ZBar_Joint: limit lower=-0.50000 upper=0.50000 effort=1000.0 velocity=0.5 -> lower=-0.50000 upper=0.00000 effort=0.00000 velocity=0.00000

Commit message: Temp fix the offset issue for now, but one of the gripper is not closing so need to fix that.

File: Testing/combined.urdf (robot description, URDF)
Before this commit: robot GantryAssembly_NoGrasper, 15 links, 14 joints
Links:
- link BasePlate: geometry collision mesh filename=C:\Users\SmorgasBORG\Documents\GitHub\FRR-Software-Interfac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 scale=1.00000 1.00000 1.00000; visual mesh filename=C:\Users\SmorgasBORG\Documents\GitHub\FRR-Software-Interfac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 scale=1.00000 1.00000 1.00000
- link CylinderCons: geometry collision mesh filename=C:\Users\SmorgasBORG\Documents\GitHub\FRR-Software-Interfac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 scale=1.00000 1.00000 1.00000; visual mesh filename=C:\Users\SmorgasBORG\Documents\GitHub\FRR-Software-Interfac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 scale=1.00000 1.00000 1.00000
- link GrasperBase: geometry collision mesh filename=C:\Users\SmorgasBORG\Documents\GitHub\FRR-Software-Interfac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 scale=1.00000 1.00000 1.00000; visual mesh filename=C:\Users\SmorgasBORG\Documents\GitHub\FRR-Software-Interfac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 scale=1.00000 1.00000 1.00000
- link LeftUpright: geometry collision mesh filename=C:\Users\SmorgasBORG\Documents\GitHub\FRR-Software-Interfac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 scale=1.00000 1.00000 1.00000; visual mesh filename=C:\Users\SmorgasBORG\Documents\GitHub\FRR-Software-Interfac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 scale=1.00000 1.00000 1.00000
- link ObjectBase: geometry collision mesh filename=C:\Users\SmorgasBORG\Documents\GitHub\FRR-Software-Interfac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 scale=1.00000 1.00000 1.00000; visual mesh filename=C:\Users\SmorgasBORG\Documents\GitHub\FRR-Software-Interfac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 scale=1.00000 1.00000 1.00000
- link RightUpright: geometry collision mesh filename=C:\Users\SmorgasBORG\Documents\GitHub\FRR-Software-Interfac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 scale=1.00000 1.00000 1.00000; visual mesh filename=C:\Users\SmorgasBORG\Documents\GitHub\FRR-Software-Interfac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 scale=1.00000 1.00000 1.00000
- link SoftJaw1: geometry collision mesh filename=C:\Users\SmorgasBORG\Documents\GitHub\FRR-Software-Interfac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 scale=1.00000 1.00000 1.00000; visual mesh filename=C:\Users\SmorgasBORG\Documents\GitHub\FRR-Software-Interfac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 scale=1.00000 1.00000 1.00000
- link SoftJaw2: geometry collision mesh filename=C:\Users\SmorgasBORG\Documents\GitHub\FRR-Software-Interfac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 scale=1.00000 1.00000 1.00000; visual mesh filename=C:\Users\SmorgasBORG\Documents\GitHub\FRR-Software-Interfac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 scale=1.00000 1.00000 1.00000
- link SoftJaw3: geometry collision mesh filename=C:\Users\SmorgasBORG\Documents\GitHub\FRR-Software-Interfac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 scale=1.00000 1.00000 1.00000; visual mesh filename=C:\Users\SmorgasBORG\Documents\GitHub\FRR-Software-Interfac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 scale=1.00000 1.00000 1.00000
- link SoftSupport1: geometry collision mesh filename=C:\Users\SmorgasBORG\Documents\GitHub\FRR-Software-Interfac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 scale=1.00000 1.00000 1.00000; visual mesh filename=C:\Users\SmorgasBORG\Documents\GitHub\FRR-Software-Interfac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 scale=1.00000 1.00000 1.00000
- link SoftSupport2: geometry collision mesh filename=C:\Users\SmorgasBORG\Documents\GitHub\FRR-Software-Interfac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 scale=1.00000 1.00000 1.00000; visual mesh filename=C:\Users\SmorgasBORG\Documents\GitHub\FRR-Software-Interfac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 scale=1.00000 1.00000 1.00000
- link SoftSupport3: geometry collision mesh filename=C:\Users\SmorgasBORG\Documents\GitHub\FRR-Software-Interfac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 scale=1.00000 1.00000 1.00000; visual mesh filename=C:\Users\SmorgasBORG\Documents\GitHub\FRR-Software-Interfac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 scale=1.00000 1.00000 1.00000
- link ZBar: geometry collision mesh filename=C:\Users\SmorgasBORG\Documents\GitHub\FRR-Software-Interfac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 scale=1.00000 1.00000 1.00000; visual mesh filename=C:\Users\SmorgasBORG\Documents\GitHub\FRR-Software-Interfac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 scale=1.00000 1.00000 1.00000
- link base_link: geometry collision mesh filename=C:\Users\SmorgasBORG\Documents\GitHub\FRR-Software-Interfac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 scale=1.00000 1.00000 1.00000; visual mesh filename=C:\Users\SmorgasBORG\Documents\GitHub\FRR-Software-Interfac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 scale=1.00000 1.00000 1.00000
- link base_link_gantry: geometry collision mesh filename=C:\Users\SmorgasBORG\Documents\GitHub\FRR-Software-Interfac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 scale=1.00000 1.00000 1.00000; visual mesh filename=C:\Users\SmorgasBORG\Documents\GitHub\FRR-Software-Interfac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 scale=1.00000 1.00000 1.00000

Commit message: Added switch for SNS retry grasp with modulation

File: Testing/combined.urdf (robot description, URDF)
Before this commit: robot GantryAssembly_NoGrasper, 15 links, 14 joints
Links:
- link BasePlate: geometry collision mesh filename=C:\Users\Ravesh\Desktop\Research\FRR\FRR Software Interface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 scale=1.00000 1.00000 1.00000; visual mesh filename=C:\Users\Ravesh\Desktop\Research\FRR\FRR Software Interface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 scale=1.00000 1.00000 1.00000
- link CylinderCons: geometry collision mesh filename=C:\Users\Ravesh\Desktop\Research\FRR\FRR Software Interface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 scale=1.00000 1.00000 1.00000; visual mesh filename=C:\Users\Ravesh\Desktop\Research\FRR\FRR Software Interface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 scale=1.00000 1.00000 1.00000
- link GrasperBase: geometry collision mesh filename=C:\Users\Ravesh\Desktop\Research\FRR\FRR Software Interface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 scale=1.00000 1.00000 1.00000; visual mesh filename=C:\Users\Ravesh\Desktop\Research\FRR\FRR Software Interface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 scale=1.00000 1.00000 1.00000
- link LeftUpright: geometry collision mesh filename=C:\Users\Ravesh\Desktop\Research\FRR\FRR Software Interface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 scale=1.00000 1.00000 1.00000; visual mesh filename=C:\Users\Ravesh\Desktop\Research\FRR\FRR Software Interface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 scale=1.00000 1.00000 1.00000
- link ObjectBase: geometry collision mesh filename=C:\Users\Ravesh\Desktop\Research\FRR\FRR Software Interface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 scale=1.00000 1.00000 1.00000; visual mesh filename=C:\Users\Ravesh\Desktop\Research\FRR\FRR Software Interface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 scale=1.00000 1.00000 1.00000
- link RightUpright: geometry collision mesh filename=C:\Users\Ravesh\Desktop\Research\FRR\FRR Software Interface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 scale=1.00000 1.00000 1.00000; visual mesh filename=C:\Users\Ravesh\Desktop\Research\FRR\FRR Software Interface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 scale=1.00000 1.00000 1.00000
- link SoftJaw1: geometry collision mesh filename=C:\Users\Ravesh\Desktop\Research\FRR\FRR Software Interface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 scale=1.00000 1.00000 1.00000; visual mesh filename=C:\Users\Ravesh\Desktop\Research\FRR\FRR Software Interface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 scale=1.00000 1.00000 1.00000
- link SoftJaw2: geometry collision mesh filename=C:\Users\Ravesh\Desktop\Research\FRR\FRR Software Interface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 scale=1.00000 1.00000 1.00000; visual mesh filename=C:\Users\Ravesh\Desktop\Research\FRR\FRR Software Interface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 scale=1.00000 1.00000 1.00000
- link SoftJaw3: geometry collision mesh filename=C:\Users\Ravesh\Desktop\Research\FRR\FRR Software Interface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 scale=1.00000 1.00000 1.00000; visual mesh filename=C:\Users\Ravesh\Desktop\Research\FRR\FRR Software Interface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 scale=1.00000 1.00000 1.00000
- link SoftSupport1: geometry collision mesh filename=C:\Users\Ravesh\Desktop\Research\FRR\FRR Software Interface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 scale=1.00000 1.00000 1.00000; visual mesh filename=C:\Users\Ravesh\Desktop\Research\FRR\FRR Software Interface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 scale=1.00000 1.00000 1.00000
- link SoftSupport2: geometry collision mesh filename=C:\Users\Ravesh\Desktop\Research\FRR\FRR Software Interface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 scale=1.00000 1.00000 1.00000; visual mesh filename=C:\Users\Ravesh\Desktop\Research\FRR\FRR Software Interface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 scale=1.00000 1.00000 1.00000
- link SoftSupport3: geometry collision mesh filename=C:\Users\Ravesh\Desktop\Research\FRR\FRR Software Interface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 scale=1.00000 1.00000 1.00000; visual mesh filename=C:\Users\Ravesh\Desktop\Research\FRR\FRR Software Interface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 scale=1.00000 1.00000 1.00000
- link ZBar: geometry collision mesh filename=C:\Users\Ravesh\Desktop\Research\FRR\FRR Software Interface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 scale=1.00000 1.00000 1.00000; visual mesh filename=C:\Users\Ravesh\Desktop\Research\FRR\FRR Software Interface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 scale=1.00000 1.00000 1.00000
- link base_link: geometry collision mesh filename=C:\Users\Ravesh\Desktop\Research\FRR\FRR Software Interface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 scale=1.00000 1.00000 1.00000; visual mesh filename=C:\Users\Ravesh\Desktop\Research\FRR\FRR Software Interface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 scale=1.00000 1.00000 1.00000
- link base_link_gantry: geometry collision mesh filename=C:\Users\Ravesh\Desktop\Research\FRR\FRR Software Interface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 scale=1.00000 1.00000 1.00000; visual mesh filename=C:\Users\Ravesh\Desktop\Research\FRR\FRR Software Interface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 scale=1.00000 1.00000 1.00000

Commit message: SNS requires a hack to set the target position x and y to be the same as the object position x and y.  Need to work with Yanjun to see if we can get rid of this.

File: Testing/combined.urdf (robot description, URDF)
Before this commit: robot GantryAssembly_NoGrasper, 15 links, 14 joints
Links:
- link BasePlate: geometry collision mesh filename=V:\Research\FRR\FRR Software Interface\FRR-Software-Interfa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 scale=1.00000 1.00000 1.00000; visual mesh filename=V:\Research\FRR\FRR Software Interface\FRR-Software-Interfa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 scale=1.00000 1.00000 1.00000
- link CylinderCons: geometry collision mesh filename=V:\Research\FRR\FRR Software Interface\FRR-Software-Interfa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 scale=1.00000 1.00000 1.00000; visual mesh filename=V:\Research\FRR\FRR Software Interface\FRR-Software-Interfa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 scale=1.00000 1.00000 1.00000
- link GrasperBase: geometry collision mesh filename=V:\Research\FRR\FRR Software Interface\FRR-Software-Interfa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 scale=1.00000 1.00000 1.00000; visual mesh filename=V:\Research\FRR\FRR Software Interface\FRR-Software-Interfa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 scale=1.00000 1.00000 1.00000
- link LeftUpright: geometry collision mesh filename=V:\Research\FRR\FRR Software Interface\FRR-Software-Interfa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 scale=1.00000 1.00000 1.00000; visual mesh filename=V:\Research\FRR\FRR Software Interface\FRR-Software-Interfa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 scale=1.00000 1.00000 1.00000
- link ObjectBase: geometry collision mesh filename=V:\Research\FRR\FRR Software Interface\FRR-Software-Interfa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 scale=1.00000 1.00000 1.00000; visual mesh filename=V:\Research\FRR\FRR Software Interface\FRR-Software-Interfa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 scale=1.00000 1.00000 1.00000
- link RightUpright: geometry collision mesh filename=V:\Research\FRR\FRR Software Interface\FRR-Software-Interfa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 scale=1.00000 1.00000 1.00000; visual mesh filename=V:\Research\FRR\FRR Software Interface\FRR-Software-Interfa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 scale=1.00000 1.00000 1.00000
- link SoftJaw1: geometry collision mesh filename=V:\Research\FRR\FRR Software Interface\FRR-Software-Interfa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 scale=1.00000 1.00000 1.00000; visual mesh filename=V:\Research\FRR\FRR Software Interface\FRR-Software-Interfa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 scale=1.00000 1.00000 1.00000
- link SoftJaw2: geometry collision mesh filename=V:\Research\FRR\FRR Software Interface\FRR-Software-Interfa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 scale=1.00000 1.00000 1.00000; visual mesh filename=V:\Research\FRR\FRR Software Interface\FRR-Software-Interfa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 scale=1.00000 1.00000 1.00000
- link SoftJaw3: geometry collision mesh filename=V:\Research\FRR\FRR Software Interface\FRR-Software-Interfa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 scale=1.00000 1.00000 1.00000; visual mesh filename=V:\Research\FRR\FRR Software Interface\FRR-Software-Interfa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 scale=1.00000 1.00000 1.00000
- link SoftSupport1: geometry collision mesh filename=V:\Research\FRR\FRR Software Interface\FRR-Software-Interfa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 scale=1.00000 1.00000 1.00000; visual mesh filename=V:\Research\FRR\FRR Software Interface\FRR-Software-Interfa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 scale=1.00000 1.00000 1.00000
- link SoftSupport2: geometry collision mesh filename=V:\Research\FRR\FRR Software Interface\FRR-Software-Interfa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 scale=1.00000 1.00000 1.00000; visual mesh filename=V:\Research\FRR\FRR Software Interface\FRR-Software-Interfa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 scale=1.00000 1.00000 1.00000
- link SoftSupport3: geometry collision mesh filename=V:\Research\FRR\FRR Software Interface\FRR-Software-Interfa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 scale=1.00000 1.00000 1.00000; visual mesh filename=V:\Research\FRR\FRR Software Interface\FRR-Software-Interfa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 scale=1.00000 1.00000 1.00000
- link ZBar: geometry collision mesh filename=V:\Research\FRR\FRR Software Interface\FRR-Software-Interfa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 scale=1.00000 1.00000 1.00000; visual mesh filename=V:\Research\FRR\FRR Software Interface\FRR-Software-Interfa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 scale=1.00000 1.00000 1.00000
- link base_link: geometry collision mesh filename=V:\Research\FRR\FRR Software Interface\FRR-Software-Interfa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 scale=1.00000 1.00000 1.00000; visual mesh filename=V:\Research\FRR\FRR Software Interface\FRR-Software-Interfa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 scale=1.00000 1.00000 1.00000
- link base_link_gantry: geometry collision mesh filename=V:\Research\FRR\FRR Software Interface\FRR-Software-Interfa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 scale=1.00000 1.00000 1.00000; visual mesh filename=V:\Research\FRR\FRR Software Interface\FRR-Software-Interfa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 scale=1.00000 1.00000 1.00000

Commit message: SNS mode doesn't close grasper, not sure why

File: Testing/combined.urdf (robot description, URDF)
Before this commit: robot GantryAssembly_NoGrasper, 15 links, 14 joints
Links:
- link BasePlate: geometry collision mesh filename=D:\Ravesh\FRR-Software-Interface\GUI\EmbeddedSystems\Gantry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 scale=1.00000 1.00000 1.00000; visual mesh filename=D:\Ravesh\FRR-Software-Interface\GUI\EmbeddedSystems\Gantry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 scale=1.00000 1.00000 1.00000
- link CylinderCons: geometry collision mesh filename=D:\Ravesh\FRR-Software-Interface\GUI\EmbeddedSystems\Gantry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 scale=1.00000 1.00000 1.00000; visual mesh filename=D:\Ravesh\FRR-Software-Interface\GUI\EmbeddedSystems\Gantry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 scale=1.00000 1.00000 1.00000
- link GrasperBase: geometry collision mesh filename=D:\Ravesh\FRR-Software-Interface\GUI\EmbeddedSystems\Gantry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 scale=1.00000 1.00000 1.00000; visual mesh filename=D:\Ravesh\FRR-Software-Interface\GUI\EmbeddedSystems\Gantry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 scale=1.00000 1.00000 1.00000
- link LeftUpright: geometry collision mesh filename=D:\Ravesh\FRR-Software-Interface\GUI\EmbeddedSystems\Gantry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 scale=1.00000 1.00000 1.00000; visual mesh filename=D:\Ravesh\FRR-Software-Interface\GUI\EmbeddedSystems\Gantry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 scale=1.00000 1.00000 1.00000
- link ObjectBase: geometry collision mesh filename=D:\Ravesh\FRR-Software-Interface\GUI\EmbeddedSystems\Gantry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 scale=1.00000 1.00000 1.00000; visual mesh filename=D:\Ravesh\FRR-Software-Interface\GUI\EmbeddedSystems\Gantry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 scale=1.00000 1.00000 1.00000
- link RightUpright: geometry collision mesh filename=D:\Ravesh\FRR-Software-Interface\GUI\EmbeddedSystems\Gantry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 scale=1.00000 1.00000 1.00000; visual mesh filename=D:\Ravesh\FRR-Software-Interface\GUI\EmbeddedSystems\Gantry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 scale=1.00000 1.00000 1.00000
- link SoftJaw1: geometry collision mesh filename=D:\Ravesh\FRR-Software-Interface\GUI\EmbeddedSystems\Gantry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 scale=1.00000 1.00000 1.00000; visual mesh filename=D:\Ravesh\FRR-Software-Interface\GUI\EmbeddedSystems\Gantry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 scale=1.00000 1.00000 1.00000
- link SoftJaw2: geometry collision mesh filename=D:\Ravesh\FRR-Software-Interface\GUI\EmbeddedSystems\Gantry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 scale=1.00000 1.00000 1.00000; visual mesh filename=D:\Ravesh\FRR-Software-Interface\GUI\EmbeddedSystems\Gantry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 scale=1.00000 1.00000 1.00000
- link SoftJaw3: geometry collision mesh filename=D:\Ravesh\FRR-Software-Interface\GUI\EmbeddedSystems\Gantry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 scale=1.00000 1.00000 1.00000; visual mesh filename=D:\Ravesh\FRR-Software-Interface\GUI\EmbeddedSystems\Gantry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 scale=1.00000 1.00000 1.00000
- link SoftSupport1: geometry collision mesh filename=D:\Ravesh\FRR-Software-Interface\GUI\EmbeddedSystems\Gantry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 scale=1.00000 1.00000 1.00000; visual mesh filename=D:\Ravesh\FRR-Software-Interface\GUI\EmbeddedSystems\Gantry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 scale=1.00000 1.00000 1.00000
- link SoftSupport2: geometry collision mesh filename=D:\Ravesh\FRR-Software-Interface\GUI\EmbeddedSystems\Gantry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 scale=1.00000 1.00000 1.00000; visual mesh filename=D:\Ravesh\FRR-Software-Interface\GUI\EmbeddedSystems\Gantry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 scale=1.00000 1.00000 1.00000
- link SoftSupport3: geometry collision mesh filename=D:\Ravesh\FRR-Software-Interface\GUI\EmbeddedSystems\Gantry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 scale=1.00000 1.00000 1.00000; visual mesh filename=D:\Ravesh\FRR-Software-Interface\GUI\EmbeddedSystems\Gantry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 scale=1.00000 1.00000 1.00000
- link ZBar: geometry collision mesh filename=D:\Ravesh\FRR-Software-Interface\GUI\EmbeddedSystems\Gantry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 scale=1.00000 1.00000 1.00000; visual mesh filename=D:\Ravesh\FRR-Software-Interface\GUI\EmbeddedSystems\Gantry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 scale=1.00000 1.00000 1.00000
- link base_link: geometry collision mesh filename=D:\Ravesh\FRR-Software-Interface\GUI\EmbeddedSystems\Gantry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 scale=1.00000 1.00000 1.00000; visual mesh filename=D:\Ravesh\FRR-Software-Interface\GUI\EmbeddedSystems\Gantry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 scale=1.00000 1.00000 1.00000
- link base_link_gantry: geometry collision mesh filename=D:\Ravesh\FRR-Software-Interface\GUI\EmbeddedSystems\Gantry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 scale=1.00000 1.00000 1.00000; visual mesh filename=D:\Ravesh\FRR-Software-Interface\GUI\EmbeddedSystems\Gantry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 scale=1.00000 1.00000 1.00000
