Commit message: Put the visualizer and render code in 2 seperate functions for modularity

File: Project_CPP/robot_arm_3/urdf/robot_arm_3.urdf (robot description, URDF)
Before this commit: robot robot_arm_3, 9 links, 8 joints
Links:
- link base_link: geometry collision mesh filename=base_link.obj; visual mesh filename=base_link.obj
- link end_eff: geometry collision mesh filename=end_eff.obj; visual mesh filename=end_eff.obj
- link l1: geometry collision mesh filename=l1.obj; visual mesh filename=l1.obj
- link l2: geometry collision mesh filename=l2.obj; visual mesh filename=l2.obj
- link l3: geometry collision mesh filename=l3.obj; visual mesh filename=l3.obj
- link l4: geometry collision mesh filename=l4.obj; visual mesh filename=l4.obj
- link l5: geometry collision mesh filename=l5.obj; visual mesh filename=l5.obj
- link l6: geometry collision mesh filename=l6.obj; visual mesh filename=l6.obj
